File: Duet2/Duet2v1.04/DuetWifi.kicad_pcb (KiCad board)
At the start: 4 copper layers, 100 x 123 mm, 351 parts, among them J1 EXPANSION, J10 E0 MOT, J11 E0 HEAT, J12 E0 TEMP, J13 E1 HEAT, J14 E1 TEMP, J15 uSDHC, J16 CONN_ALT_HEADER, J19 Z_STOP, J2 FAN2, J20 5V_PS, J21 JTAG, J22 USB, J23 VIN, J24 GND V_IN, J25 FAN0, J28 Probe, J29 FAN1, J3 5V V_FAN VIN, J30 PanelDUE, J31 GND V_IN, J32 Y_STOP, J33 X_STOP, J34 E0_STOP, J35 E1_STOP, J36 Z A, J37 SPI0, J39 ESP_COMMS, J4 BED HEAT, J5 BED TEMP, J6 E1 MOT, J7 Z B, J8 Y MOT, J9 X MOT, M1 FID, M10 CE Logo, M2 FID, M3 FID, M4 MOUNTING, M5 MOUNTING, M6 MOUNTING, M7 MOUNTING, M8 LOGO, M9 CE Logo, P1 CONN_SD, P2 CONN_LCD, U1 ATSAM4E8E, U10 74HC125, U11 74HCT02, U12 74HC74, U13 74HC32, U2 AP7361C-33E-13, U3 A4403, U4 ESP-07/12, U5 TMC2660, U6 TMC2660, U7 TMC2660, U8 TMC2660, U9 TMC2660, X2 CRYSTAL_4PIN

Commit message: Add files via upload
Parts:
- removed D4: Diag, complib:D_0603
- removed L4: MFB-201209-0011PW, complib:R_0805
- removed M10: CE Logo, complib:Logo_CE_5mm_mirror
- removed M9: CE Logo, complib:Logo_CE_5mm
- removed R104: 2K2, complib:R_0603
- removed R92: 3R3 0.33W, complib:R_0805
- removed R94: 0R051, complib:R_1206
- removed TP1, TP5: Z_Stp_Tp, complib:CONN_3x1
- removed TP15: TP, complib:TP_via
- removed TP2: Y_Stp_Tp, complib:CONN_3x1
- removed TP3: X_Stp_Tp, complib:CONN_3x1
- removed TP4: E0_Stp_Tp, complib:CONN_3x1
- added C112: 0u1 16V, complib:C_0603, B.Cu at (91.5, 112.4)
- added C126: 10n/100n, complib:C_0603, B.Cu at (101.3, 130.6)
- added C127: 0u1 16V, complib:C_0603, B.Cu at (92.1, 78.4)
- added C128: 0u1 16V, complib:C_0603, B.Cu at (92.8, 95.1)
- added C129: 0u1 16V, complib:C_0603, B.Cu at (91.8, 88.0)
- added C130: 0u1 16V, complib:C_0603, B.Cu at (92.2, 104.7)
- added C131: 0u1 16V, complib:C_0603, B.Cu at (92.7, 62.8)
- added C132: 0u1 16V, complib:C_0603, B.Cu at (92.5, 72.4)
- added C133: 0u1 16V, complib:C_0603, B.Cu at (95.3, 45.0)
- added C134: 0u1 16V, complib:C_0603, B.Cu at (95.1, 54.6)
- added C92: 2u2, complib:C_0603, B.Cu at (99.9, 111.9)
- added C93: 22n X7R 10% 16V, complib:C_0603, B.Cu at (102.0, 121.3)
- added C95: 0u1 50V, complib:C_0603, B.Cu at (97.7, 112.7)
- added J17: + + - -, complib:PIN_ARRAY_4x1, F.Cu at (90.2, 130.2)
- added J18: + + - -, complib:PIN_ARRAY_4x1, F.Cu at (105.0, 130.2)
- added J26: E2/E3_UART, complib:PIN_ARRAY_2X1_mod, F.Cu at (112.3, 134.5)
- added J27: UART, complib:tp_smd, F.Cu at (108.1, 80.8)
- added J38: ENN, complib:tp_smd, F.Cu at (108.2, 84.3)
- added J40: DIR, complib:tp_smd, F.Cu at (108.1, 81.9)
- added J41: STEP, complib:tp_smd, F.Cu at (108.2, 83.1)
- added J42: UART, complib:tp_smd, F.Cu at (107.0, 65.6)
- added J43: ENN, complib:tp_smd, F.Cu at (107.0, 68.1)
- added J44: DIR, complib:tp_smd, F.Cu at (107.0, 66.9)
- added J45: STEP, complib:tp_smd, F.Cu at (107.0, 69.4)
- added J46: UART, complib:tp_smd, F.Cu at (110.2, 46.8)
- added J47: ENN, complib:tp_smd, F.Cu at (110.2, 49.3)
- added J48: DIR, complib:tp_smd, F.Cu at (110.2, 48.1)
- added J49: STEP, complib:tp_smd, F.Cu at (110.2, 50.6)
- added J50: UART, complib:tp_smd, F.Cu at (107.4, 97.3)
- added J51: ENN, complib:tp_smd, F.Cu at (107.4, 100.0)
- added J52: DIR, complib:tp_smd, F.Cu at (107.4, 98.6)
- added J53: STEP, complib:tp_smd, F.Cu at (107.4, 101.3)
- added J54: UART, complib:tp_smd, F.Cu at (106.9, 113.7)
- added J55: ENN, complib:tp_smd, F.Cu at (106.9, 116.9)
- added J56: DIR, complib:tp_smd, F.Cu at (106.9, 115.1)
- added J57: STEP, complib:tp_smd, F.Cu at (106.9, 118.2)
- added Ju1: 2, complib:R_0603, F.Cu at (94.4, 127.6)
- added Ju2: 2/3, complib:R_0603, F.Cu at (94.4, 133.5)
- added Ju3: 2/3, complib:R_0603, B.Cu at (102.9, 133.5)
- added Ju4: 2, complib:R_0603, B.Cu at (102.9, 127.8)
- added L10: 50R@100MHz, Inductor_SMD:L_1206_3216Metric_Pad1.42x1.75mm_HandSolder, B.Cu at (91.4, 82.0)
- added L11: 50R@100MHz, Inductor_SMD:L_1206_3216Metric_Pad1.42x1.75mm_HandSolder, B.Cu at (91.4, 76.6)
- added L12: 50R@100MHz, Resistor_SMD:R_1206_3216Metric_Pad1.42x1.75mm_HandSolder, B.Cu at (92.6, 68.7)
- added L13: 50R@100MHz, Resistor_SMD:R_1206_3216Metric_Pad1.42x1.75mm_HandSolder, B.Cu at (91.7, 74.3)
- added L14: 50R@100MHz, Resistor_SMD:R_1206_3216Metric_Pad1.42x1.75mm_HandSolder, B.Cu at (92.6, 66.5)
- added L15: 50R@100MHz, Resistor_SMD:R_1206_3216Metric_Pad1.42x1.75mm_HandSolder, B.Cu at (92.5, 60.9)
- added L16: 50R@100MHz, Resistor_SMD:R_1206_3216Metric_Pad1.42x1.75mm_HandSolder, B.Cu at (95.1, 50.9)
- added L17: 50R@100MHz, Resistor_SMD:R_1206_3216Metric_Pad1.42x1.75mm_HandSolder, B.Cu at (95.3, 56.4)
- added L18: 50R@100MHz, Resistor_SMD:R_1206_3216Metric_Pad1.42x1.75mm_HandSolder, B.Cu at (95.1, 48.6)
- added L19: 50R@100MHz, Resistor_SMD:R_1206_3216Metric_Pad1.42x1.75mm_HandSolder, B.Cu at (96.6, 43.1)
- added L20: 50R@100MHz, Resistor_SMD:R_1206_3216Metric_Pad1.42x1.75mm_HandSolder, B.Cu at (92.1, 101.0)
- added L21: 50R@100MHz, Resistor_SMD:R_1206_3216Metric_Pad1.42x1.75mm_HandSolder, B.Cu at (92.3, 106.6)
- added L22: 50R@100MHz, Resistor_SMD:R_1206_3216Metric_Pad1.42x1.75mm_HandSolder, B.Cu at (92.1, 98.7)
- added L23: 50R@100MHz, Resistor_SMD:R_1206_3216Metric_Pad1.42x1.75mm_HandSolder, B.Cu at (93.3, 93.2)
- added L24: 50R@100MHz, Resistor_SMD:R_1206_3216Metric_Pad1.42x1.75mm_HandSolder, B.Cu at (91.7, 118.2)
- added L25: 50R@100MHz, Resistor_SMD:R_1206_3216Metric_Pad1.42x1.75mm_HandSolder, B.Cu at (91.8, 124.1)
- added L26: 50R@100MHz, Resistor_SMD:R_1206_3216Metric_Pad1.42x1.75mm_HandSolder, B.Cu at (91.7, 116.0)
- added L27: 50R@100MHz, Resistor_SMD:R_1206_3216Metric_Pad1.42x1.75mm_HandSolder, B.Cu at (92.3, 110.6)
- added L8: 50R@100MHz, Inductor_SMD:L_1206_3216Metric_Pad1.42x1.75mm_HandSolder, B.Cu at (91.5, 84.3)
- added L9: 50R@100MHz, Resistor_SMD:R_1206_3216Metric_Pad1.42x1.75mm_HandSolder, B.Cu at (92.0, 89.9)
- added M11: LOGO, Symbol:Untitled, B.Cu at (147.3, 131.7)
- added U16: SN74CB3Q3251, complib:QSOP-16_3.9x4.9mm_Pitch0.635mm, F.Cu at (112.0, 130.4)
- added VR1: 3J, Inductor_THT:L_1812_HandSoldering, F.Cu at (91.4, 79.1)
- added VR10: 3J, Inductor_THT:L_1812_HandSoldering, F.Cu at (84.3, 59.0)
- added VR11: 3J, Inductor_THT:L_1812_HandSoldering, F.Cu at (91.4, 72.8)
- added VR12: 3J, Inductor_THT:L_1812_HandSoldering, B.Cu at (87.9, 63.2)
- added VR13: 3J, Inductor_THT:L_1812_HandSoldering, F.Cu at (95.2, 53.7)
- added VR14: 3J, Inductor_THT:L_1812_HandSoldering, B.Cu at (85.6, 58.0)
- added VR15: 3J, Inductor_THT:L_1812_HandSoldering, B.Cu at (86.6, 52.6)
- added VR16: 3J, Inductor_THT:L_1812_HandSoldering, B.Cu at (90.5, 40.3)
- added VR17: 3J, Inductor_THT:L_1812_HandSoldering, F.Cu at (95.3, 46.3)
- added VR18: 3J, Inductor_THT:L_1812_HandSoldering, B.Cu at (95.8, 40.0)
- added VR19: 3J, Inductor_THT:L_1812_HandSoldering, F.Cu at (91.1, 95.4)
- added VR2: 3J, Inductor_THT:L_1812_HandSoldering, F.Cu at (91.4, 83.8)
- added VR20: 3J, Inductor_THT:L_1812_HandSoldering, F.Cu at (91.1, 100.1)
- added VR21: 3J, Inductor_THT:L_1812_HandSoldering, B.Cu at (87.6, 103.4)
- added VR22: 3J, Inductor_THT:L_1812_HandSoldering, F.Cu at (84.0, 92.1)
- added VR23: 3J, Inductor_THT:L_1812_HandSoldering, F.Cu at (91.1, 105.5)
- added VR24: 3J, Inductor_THT:L_1812_HandSoldering, B.Cu at (88.8, 94.2)
- added VR25: 3J, Inductor_THT:L_1812_HandSoldering, F.Cu at (91.2, 112.6)
- added VR26: 3J, Inductor_THT:L_1812_HandSoldering, F.Cu at (91.2, 117.3)
- added VR27: 3J, Inductor_THT:L_1812_HandSoldering, B.Cu at (87.3, 119.6)
- added VR28: 3J, Inductor_THT:L_1812_HandSoldering, F.Cu at (83.9, 109.2)
- added VR29: 3J, Inductor_THT:L_1812_HandSoldering, F.Cu at (91.3, 122.4)
- added VR3: 3J, Inductor_THT:L_1812_HandSoldering, B.Cu at (86.7, 86.8)
- added VR30: 3J, Inductor_THT:L_1812_HandSoldering, B.Cu at (88.2, 111.7)
- added VR4: 3J, Inductor_THT:L_1812_HandSoldering, F.Cu at (83.9, 75.8)
- added VR5: 3J, Inductor_THT:L_1812_HandSoldering, F.Cu at (91.4, 88.7)
- added VR6: 3J, Inductor_THT:L_1812_HandSoldering, B.Cu at (86.6, 78.8)
- added VR7: 3J, Inductor_THT:L_1812_HandSoldering, F.Cu at (91.4, 62.4)
- added VR8: 3J, Inductor_THT:L_1812_HandSoldering, F.Cu at (91.3, 67.4)
- added VR9: 3J, Inductor_THT:L_1812_HandSoldering, B.Cu at (86.7, 69.8)
- C100: value 0u47 -> 0.1u 50V; moved to B.Cu
- C101, C75, C76, C77, C78: value 1u 50V -> 0u1 50V; moved to B.Cu
- C103: value 0u1 50V -> 0u1
- C104, C24, C25, C35, C37: moved to B.Cu
- C105: value 0u01 X7R 10% 50V -> 10n/100n
- C106, C107, C108, C109, C113, C114, C115, C116, C117, C118, C119, C120, C121, C122, C123, C85, C86, C87, C88, C89: value 1n >50V -> 470p 100V; moved to B.Cu
- C110: value 0u01 X7R 10% 50V -> 2n2; moved to B.Cu
- C124: value 0u1 -> 0u1 16V; moved to B.Cu
- C14, C56: value 0u01 X7R 10% 50V -> 0u1 50V; moved to B.Cu
- C15, C28, C38: value 0u01 X7R 10% 50V -> 2u2; moved to B.Cu
- C20, C21, C30: value 0u47 -> 22n X7R 10% 16V; moved to B.Cu
- C26, C27, C36: value 0u1 -> 0.1u 50V; moved to B.Cu
- C29: value 0u01 X7R 10% 50V -> 0u1; moved to B.Cu
- C31: value 0u47 -> 2u2; moved to B.Cu
- C34: value 0u1 50V -> 0u1; moved to B.Cu
- C39: value 0u01 X7R 10% 50V -> 22n X7R 10% 16V; moved to B.Cu
- C55: value 0u1 -> 2n2
- C57: value 0u01 X7R 10% 50V -> 0.1u 50V; moved to B.Cu
- C99: value 220u 10V -> 220u 25V
- L5, L6: footprint complib:R_0603 -> complib:R_0805_extended_pads
- R107: value 10K -> 100R
- R26, R89: value 22R -> 22K; moved to B.Cu
- R27, R29, R39, R41, R90: value 22R -> 0R075 1% 0.33W; footprint complib:R_0603 -> complib:R_0805_extended_pads; moved to B.Cu
- R28: value 22R -> 1K
- R30: value 68R -> 3k9; moved to B.Cu
- R32, R33, R44, R45, R93: value 0R051 -> 0R075 1% 0.33W; footprint complib:R_1206 -> complib:R_0805_extended_pads; moved to B.Cu
- R34: value 0R051 -> 10M; footprint complib:R_1206 -> complib:R_0603; moved to B.Cu
- R35, R46, R47: value 0R051 -> 22K; footprint complib:R_1206 -> complib:R_0603; moved to B.Cu
- R38: value 22R -> 3k9
- R40: value 22R -> 10M
- R85, R86: footprint complib:R_0805 -> complib:R_1206
- R87: value 3K92 -> 3K6
- R88: value 750R -> 680R
- TR4: footprint FE Footprints:D-PAK -> Symbol:D-PAK
- U10: value 74HC125 -> MAX31865AAP(SSOP20); footprint complib:TSSOP-14 -> complib:QFN-20-1EP_5x5mm_Pitch0.65mm_mod
- U11: footprint FE Footprints:TSSOP-14 -> complib:TSSOP-14
- U13: value 74HC32 -> MAX31865AAP(SSOP20); footprint complib:TSSOP-14 -> complib:QFN-20-1EP_5x5mm_Pitch0.65mm_mod; moved to B.Cu
- U5, U6, U7, U8, U9: value TMC2660 -> TMC2224; footprint FE Footprints:TMC2660 -> complib:QFN-28-1EP_5x5mm_Pitch0.5mm; moved to B.Cu
- moved R28 82.4 mm to (109.9, 125.0), turned to 0 degrees
- moved U9 75.9 mm to (103.1, 49.4), turned to 90 degrees
- moved U6 66.8 mm to (100.1, 116.7), turned to 90 degrees
- moved R38 62.0 mm to (99.7, 125.9), turned to 180 degrees
- moved U10 50.8 mm to (98.9, 129.6), turned to 270 degrees
- moved R30 49.6 mm to (96.3, 125.9)
- moved R34 46.6 mm to (99.4, 125.9)
- moved C55 41.2 mm to (102.4, 124.0)
- moved D10 39.9 mm to (114.9, 80.9), turned to 90 degrees
- moved U8 39.3 mm to (100.2, 67.4), turned to 90 degrees
- moved D9 36.4 mm to (116.7, 87.4), turned to 90 degrees
- moved R70 35.8 mm to (114.9, 77.9), turned to 90 degrees
- moved D19 35.6 mm to (116.7, 118.7), turned to 90 degrees
- moved D12 34.8 mm to (116.9, 97.7), turned to 90 degrees
- moved D11 34.5 mm to (116.7, 109.8)
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Connections:
- C100 pad 1: Net-(C100-Pad1) -> V_FUSED
- C100 pad 2: GND -> Net-(C100-Pad2)
- C103 pad 1: V_FUSED -> GND
- C103 pad 2: Net-(C103-Pad2) -> +3.3V
- C105 pad 2: GND -> Net-(C105-Pad2)
- C107 pad 1: GND -> X_MOT_2A
- C107 pad 2: X_MOT_2A -> GND
- C108 pad 1: GND -> Y_MOT_2A
- C108 pad 2: Y_MOT_2A -> GND
- C109 pad 1: GND -> Z_MOT_2A
- C109 pad 2: Z_MOT_2A -> GND
- C110 pad 1: Net-(C110-Pad1) -> +3.3V
- C113 pad 1: GND -> X_MOT_2B
- C113 pad 2: X_MOT_2B -> GND
- C114 pad 1: GND -> Y_MOT_2B
- C114 pad 2: Y_MOT_2B -> GND
- C115 pad 1: GND -> Z_MOT_2B
- C115 pad 2: Z_MOT_2B -> GND
- C116 pad 1: GND -> E0_MOT_1B
- C116 pad 2: E0_MOT_1B -> GND
- C117 pad 1: GND -> E1_MOT_1B
- C117 pad 2: E1_MOT_1B -> GND
- C118 pad 1: GND -> E0_MOT_1A
- C118 pad 2: E0_MOT_1A -> GND
- C119 pad 1: GND -> E1_MOT_1A
- C119 pad 2: E1_MOT_1A -> GND
- C124 pad 1: +3.3V -> GND
- C124 pad 2: GND -> Net-(C124-Pad2)
- C14 pad 1: Net-(C14-Pad1) -> +3.3V
- C20 pad 2: GND -> Net-(C20-Pad2)
- C21 pad 2: GND -> Net-(C21-Pad2)
- C24 pad 2: Net-(C24-Pad2) -> GND
- C25 pad 2: Net-(C25-Pad2) -> GND
- C26 pad 1: +3.3V -> V_FUSED
- C26 pad 2: GND -> Net-(C26-Pad2)
- C27 pad 1: +3.3V -> V_FUSED
- C27 pad 2: GND -> Net-(C27-Pad2)
- C29 pad 1: Net-(C29-Pad1) -> +3.3V
- C30 pad 2: GND -> Net-(C30-Pad2)
- C31 pad 1: Net-(C31-Pad1) -> GND
- C31 pad 2: GND -> Net-(C31-Pad2)
- C34 pad 1: V_FUSED -> +3.3V
- C34 pad 2: Net-(C34-Pad2) -> GND
- C35 pad 2: Net-(C35-Pad2) -> GND
- C36 pad 1: +3.3V -> V_FUSED
- C36 pad 2: GND -> Net-(C36-Pad2)
- C39 pad 2: GND -> Net-(C39-Pad2)
- C56 pad 1: Net-(C56-Pad1) -> V_FUSED
- C57 pad 1: Net-(C57-Pad1) -> V_FUSED
- C57 pad 2: GND -> Net-(C57-Pad2)
- J1 pad 32: SPI1_SCK_BUFF_EXP -> MOT_TXD
- J1 pad 33: SPI1_MOSI_BUFF -> +5V
- J1 pad 34: SPI1_MISO -> MOT_RXD
- J21 pad 6: PB5/TDO -> MUX_1
- J21 pad 7: (no net) -> Net-(J21-Pad7)
- J21 pad 8: PB4/TDI -> TEMP_CS2
- J22 pad 4: (no net) -> Net-(J22-Pad4)
- J37 pad 10: (no net) -> Net-(J37-Pad10)
- R26 pad 1: Net-(R26-Pad1) -> X_UART
- R26 pad 2: Net-(C14-Pad1) -> +3.3V
- R27 pad 1: Net-(R27-Pad1) -> GND
- R27 pad 2: Net-(C28-Pad1) -> Net-(C127-Pad2)
- R28 pad 1: Net-(R28-Pad1) -> MOT_RXD
- R28 pad 2: Net-(C15-Pad1) -> MOT_TXD
- R29 pad 1: Net-(R29-Pad1) -> GND
- R29 pad 2: Net-(C29-Pad1) -> Net-(C133-Pad2)
- R30 pad 1: SPI1_SCK_BUFF -> Net-(R30-Pad1)
- R30 pad 2: SPI1_SCK_BUFF_EXP -> Net-(R30-Pad2)
- R32 pad 2: Net-(R27-Pad1) -> Net-(C129-Pad2)
- R33 pad 2: Net-(R29-Pad1) -> Net-(C134-Pad2)
- R34 pad 1: GND -> Net-(R30-Pad1)
- R34 pad 2: Net-(R26-Pad1) -> Net-(C126-Pad2)
- R35 pad 1: GND -> Z_UART
- R35 pad 2: Net-(R28-Pad1) -> +3.3V
- R36 pad 2: PB4/TDI -> TEMP_CS2
- R38 pad 2: Net-(C38-Pad1) -> Net-(R38-Pad2)
- R39 pad 1: Net-(R39-Pad1) -> GND
- R39 pad 2: Net-(C56-Pad1) -> Net-(C131-Pad2)
- R40 pad 1: Net-(R40-Pad1) -> Net-(R38-Pad1)
- R40 pad 2: Net-(C39-Pad1) -> Net-(C105-Pad2)
- R41 pad 1: Net-(R41-Pad1) -> GND
- R41 pad 2: Net-(C57-Pad1) -> Net-(C130-Pad2)
- R44 pad 2: Net-(R39-Pad1) -> Net-(C132-Pad2)
- R45 pad 2: Net-(R41-Pad1) -> Net-(C128-Pad2)
- R46 pad 1: GND -> Y_UART
- R46 pad 2: Net-(R38-Pad1) -> +3.3V
- R47 pad 1: GND -> E0_UART
- R47 pad 2: Net-(R40-Pad1) -> +3.3V
- R89 pad 1: Net-(R89-Pad1) -> +3.3V
- R89 pad 2: Net-(C105-Pad1) -> E1_UART
- R90 pad 1: Net-(R90-Pad1) -> Net-(C112-Pad2)
- R90 pad 2: Net-(C110-Pad1) -> GND
- R93 pad 1: GND -> Net-(C124-Pad2)
- R93 pad 2: Net-(R90-Pad1) -> GND
- U1 pad 103: E0_EN -> TEMP_MISO
- U1 pad 105: PB4/TDI -> TEMP_CS2
- U1 pad 109: PB5/TDO -> MUX_1
- U1 pad 133: E1_EN -> MUX_0
- U1 pad 32: SPI1_MISO -> MOT_RXD
- U1 pad 37: SPI1_MOSI -> MOT_TXD
- U1 pad 46: SPI1_SCK -> TEMP_SCK
- U1 pad 84: X_EN -> TEMP_CS1
- U1 pad 86: Y_EN -> MUX_2
- U1 pad 90: Z_EN -> TEMP_MOSI
- U10 pad 1: GND -> Net-(R38-Pad1)
- U10 pad 11: SPI1_MOSI_BUFF -> TEMP_MOSI
- U10 pad 12: SPI1_MOSI -> TEMP_SCK
- U10 pad 13: GND -> TEMP_CS1
- U10 pad 14: +3.3V -> TEMP_MISO
- U10 pad 2: SPI1_SCK -> Net-(R38-Pad1)
- U10 pad 3: SPI1_SCK_BUFF_EXP -> Net-(R38-Pad2)
- U10 pad 4: GND -> Net-(R38-Pad2)
- U10 pad 5: Z_PROBE_MOD -> Net-(J17-Pad4)
- U10 pad 6: Z_PROBE_MOD_BUFF -> Net-(J17-Pad4)
- U10 pad 7: GND -> Net-(C105-Pad2)
- U10 pad 8: (no net) -> Net-(C105-Pad1)
- U10 pad 9: GND -> Net-(J17-Pad1)
- U12 pad 6: (no net) -> Net-(U12-Pad6)
- U12 pad 8: (no net) -> Net-(U12-Pad8)
- U12 pad 9: (no net) -> Net-(U12-Pad9)
- U13 pad 1: SG_TST_X -> Net-(R30-Pad1)
- U13 pad 10: Net-(U13-Pad10) -> GND
- U13 pad 11: PB5/TDO -> TEMP_MOSI
- U13 pad 12: Net-(U13-Pad12) -> TEMP_SCK
- U13 pad 13: Net-(U13-Pad13) -> TEMP_CS2
- U13 pad 14: +3.3V -> TEMP_MISO
- U13 pad 2: SG_TST_Y -> Net-(R30-Pad1)
- U13 pad 3: Net-(U13-Pad10) -> Net-(R30-Pad2)
- U13 pad 4: SG_TST_Z -> Net-(R30-Pad2)
- U13 pad 5: SG_TST_E1 -> Net-(J18-Pad4)
- U13 pad 6: Net-(U13-Pad12) -> Net-(J18-Pad4)
- U13 pad 7: GND -> Net-(C126-Pad2)
- U13 pad 8: Net-(U13-Pad13) -> Net-(C126-Pad1)
- U13 pad 9: SG_TST_E0 -> Net-(J18-Pad1)
- U3 pad 1: Net-(L4-Pad1) -> Net-(C12-Pad1)
- U5 pad 1: V_FUSED -> GND
- U5 pad 12: Net-(C14-Pad1) -> Net-(C128-Pad2)
- U5 pad 13: Net-(C20-Pad1) -> Net-(L23-Pad2)
- U5 pad 14: SPI1_MISO -> V_FUSED
- U5 pad 15: SPI1_MOSI_BUFF -> GND
- U5 pad 16: SPI1_SCK_BUFF -> GND
- U5 pad 18: X_EN -> Net-(C31-Pad2)
- U5 pad 19: ENN -> +3.3V
- U5 pad 20: (no net) -> E0_UART
- U5 pad 21: GND -> Net-(U5-Pad21)
- U5 pad 22: Net-(C28-Pad1) -> GND
- U5 pad 25: Net-(R27-Pad1) -> E0_STEP
- U5 pad 4: V_FUSED -> Net-(C39-Pad2)
- U5 pad 9: Net-(R26-Pad1) -> Net-(C130-Pad2)
- U6 pad 1: V_FUSED -> GND
- U6 pad 12: Net-(C15-Pad1) -> Net-(C112-Pad2)
- U6 pad 13: Net-(C21-Pad1) -> Net-(L27-Pad2)
- U6 pad 14: SPI1_MISO -> V_FUSED
- U6 pad 15: SPI1_MOSI_BUFF -> GND
- U6 pad 16: SPI1_SCK_BUFF -> GND
- U6 pad 18: Z_EN -> Net-(C92-Pad1)
- U6 pad 19: ENN -> +3.3V
- U6 pad 20: (no net) -> E1_UART
- U6 pad 21: GND -> Net-(U6-Pad21)
- U6 pad 22: Net-(C29-Pad1) -> GND
- U6 pad 25: Net-(R29-Pad1) -> E1_STEP
- U6 pad 4: V_FUSED -> Net-(C93-Pad1)
- U6 pad 9: Net-(R28-Pad1) -> Net-(C124-Pad2)
- U7 pad 1: V_FUSED -> GND
- U7 pad 12: Net-(C38-Pad1) -> Net-(C127-Pad2)
- U7 pad 13: Net-(C30-Pad1) -> Net-(L11-Pad2)
- U7 pad 14: SPI1_MISO -> V_FUSED
- U7 pad 15: SPI1_MOSI_BUFF -> GND
- U7 pad 16: SPI1_SCK_BUFF -> GND
- U7 pad 18: Y_EN -> Net-(C28-Pad1)
- U7 pad 19: ENN -> +3.3V
- U7 pad 20: (no net) -> X_UART
- U7 pad 21: GND -> Net-(U7-Pad21)
- U7 pad 22: Net-(C56-Pad1) -> GND
- U7 pad 25: Net-(R39-Pad1) -> X_STEP
- U7 pad 4: V_FUSED -> Net-(C20-Pad2)
- U7 pad 9: Net-(R38-Pad1) -> Net-(C129-Pad2)
- U8 pad 1: V_FUSED -> GND
- U8 pad 12: Net-(C39-Pad1) -> Net-(C131-Pad2)
- U8 pad 13: Net-(C31-Pad1) -> Net-(L15-Pad2)
- U8 pad 14: SPI1_MISO -> V_FUSED
- U8 pad 15: SPI1_MOSI_BUFF -> GND
- U8 pad 16: SPI1_SCK_BUFF -> GND
- U8 pad 18: E0_EN -> Net-(C38-Pad1)
- U8 pad 19: ENN -> +3.3V
- U8 pad 20: (no net) -> Y_UART
- U8 pad 21: GND -> Net-(U8-Pad21)
- U8 pad 22: Net-(C57-Pad1) -> GND
- U8 pad 25: Net-(R41-Pad1) -> Y_STEP
- U8 pad 4: V_FUSED -> Net-(C30-Pad2)
- U8 pad 9: Net-(R40-Pad1) -> Net-(C132-Pad2)
- U9 pad 1: V_FUSED -> GND
- U9 pad 12: Net-(C105-Pad1) -> Net-(C133-Pad2)
- U9 pad 13: Net-(C100-Pad1) -> Net-(L19-Pad2)
- U9 pad 14: SPI1_MISO -> V_FUSED
- U9 pad 15: SPI1_MOSI_BUFF -> GND
- U9 pad 16: SPI1_SCK_BUFF -> GND
- U9 pad 18: E1_EN -> Net-(C15-Pad1)
- U9 pad 19: ENN -> +3.3V
- U9 pad 20: (no net) -> Z_UART
- U9 pad 21: GND -> Net-(U9-Pad21)
- U9 pad 22: Net-(C110-Pad1) -> GND
- U9 pad 25: Net-(R90-Pad1) -> Z_STEP
- U9 pad 4: V_FUSED -> Net-(C21-Pad2)
- U9 pad 9: Net-(R89-Pad1) -> Net-(C134-Pad2)
Routing:
- net V_FUSED: track 252.4 -> 1280.9 mm, vias 8 -> 58
- net GND: track 476.3 -> 771.2 mm, vias 171 -> 218
- net SPI1_MISO: track 260.4 -> 0.00 mm, vias 9 -> 0
- net SPI1_MOSI_BUFF: track 234.6 -> 0.00 mm, vias 9 -> 0
- net SPI1_SCK_BUFF: track 172.9 -> 0.00 mm, vias 7 -> 0
- net MOT_TXD: track 0.00 -> 148.1 mm, vias 0 -> 9
- net MOT_RXD: track 0.00 -> 119.9 mm, vias 0 -> 5
- net Z_UART: track 0.00 -> 113.1 mm, vias 0 -> 3
- net TEMP_SCK: track 0.00 -> 110.3 mm, vias 0 -> 7
- net SG_TST_Z: track 109.4 -> 0.00 mm, vias 4 -> 0
- net Z_PROBE_MOD_BUFF: track 100.9 -> 0.00 mm, vias 2 -> 0
- net Z_EN: track 99.7 -> 0.00 mm, vias 2 -> 0
- net Y_UART: track 0.00 -> 99.1 mm, vias 0 -> 3
- net TEMP_CS2: track 0.00 -> 92.6 mm, vias 0 -> 7
- net SG_TST_Y: track 87.6 -> 0.00 mm, vias 5 -> 0
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- removed copper zone on B.Cu, net E0_MOT_1A
- removed copper zone on F.Cu, net E0_MOT_1A
- removed copper zone on B.Cu, net E0_MOT_1B
- removed copper zone on F.Cu, net E0_MOT_1B
- removed copper zone on B.Cu, net E0_MOT_2A
- removed copper zone on F.Cu, net E0_MOT_2A
- removed copper zone on B.Cu, net E0_MOT_2B
- removed copper zone on F.Cu, net E0_MOT_2B
- removed copper zone on B.Cu, net E1_MOT_1A
- removed copper zone on F.Cu, net E1_MOT_1A
- removed copper zone on B.Cu, net E1_MOT_1B
- removed copper zone on F.Cu, net E1_MOT_1B
- removed copper zone on B.Cu, net E1_MOT_2A
- removed copper zone on F.Cu, net E1_MOT_2A
- removed copper zone on B.Cu, net E1_MOT_2B
- removed copper zone on F.Cu, net E1_MOT_2B
- removed copper zone on F.Cu, net Net-(R26-Pad1)
- removed copper zone on F.Cu, net Net-(R27-Pad1)
- removed copper zone on F.Cu, net Net-(R28-Pad1)
- removed copper zone on F.Cu, net Net-(R29-Pad1)
- removed copper zone on F.Cu, net Net-(R38-Pad1)
- removed copper zone on F.Cu, net Net-(R39-Pad1)
- removed copper zone on F.Cu, net Net-(R40-Pad1)
- removed copper zone on F.Cu, net Net-(R41-Pad1)
- removed copper zone on F.Cu, net Net-(R89-Pad1)
- removed copper zone on F.Cu, net Net-(R90-Pad1)
- removed copper zone on F.Cu, net V_FUSED
- removed copper zone on B.Cu, net X_MOT_1A
- removed copper zone on F.Cu, net X_MOT_1A
- removed copper zone on B.Cu, net X_MOT_1B
- removed copper zone on F.Cu, net X_MOT_1B
- removed copper zone on B.Cu, net X_MOT_2A
- removed copper zone on F.Cu, net X_MOT_2A
- removed copper zone on B.Cu, net X_MOT_2B
- removed copper zone on F.Cu, net X_MOT_2B
- removed copper zone on B.Cu, net Y_MOT_1A
- removed copper zone on F.Cu, net Y_MOT_1A
- removed copper zone on B.Cu, net Y_MOT_1B
- removed copper zone on F.Cu, net Y_MOT_1B
- removed copper zone on B.Cu, net Y_MOT_2A
- removed copper zone on F.Cu, net Y_MOT_2A
- removed copper zone on B.Cu, net Y_MOT_2B
- removed copper zone on F.Cu, net Y_MOT_2B
- removed copper zone on B.Cu, net Z_MOT_1A
- removed copper zone on F.Cu, net Z_MOT_1A
- removed copper zone on B.Cu, net Z_MOT_1B
- removed copper zone on F.Cu, net Z_MOT_1B
- removed copper zone on B.Cu, net Z_MOT_2A
- removed copper zone on F.Cu, net Z_MOT_2A
- removed copper zone on B.Cu, net Z_MOT_2B
- removed copper zone on F.Cu, net Z_MOT_2B
Other:
- net class 0.2 added: clearance 0.2, trace_width 0.2, via_dia 0.6, via_drill 0.4
- net class 0.25 added: clearance 0.2, trace_width 0.25, via_dia 0.6, via_drill 0.4
- net class 0.254 removed
- net class 0.29 added: clearance 0.2, trace_width 0.29, via_dia 0.6, via_drill 0.4
- net class 0.4455 removed
- net class 0.5 added: clearance 0.25, trace_width 0.5, via_dia 0.8, via_drill 0.5
- net class 0.508 removed
- net class 0.75 added: clearance 0.25, trace_width 0.75, via_dia 0.8, via_drill 0.5
- net class 0.762 removed
- net class 1 added: clearance 0.25, trace_width 1, via_dia 0.8, via_drill 0.5
- net class 1.016 removed
- net class 1.5 added: clearance 0.25, trace_width 1.5, via_dia 0.8, via_drill 0.5
- net class 1.524 removed
- net class 1.778 removed
- net class 2.0 added: clearance 0.25, trace_width 2, via_dia 0.9, via_drill 0.6
- net class 2.032 removed
- net class 2.286 removed
- net class 2.5 added: clearance 0.25, trace_width 2.5, via_dia 0.9, via_drill 0.6
- net class 2.54 removed
- net class 3.5 added: clearance 0.25, trace_width 3.5, via_dia 0.9, via_drill 0.6
- net class 3.81 removed
- net class Default: trace_width 0.254 -> 0.25; via_dia 0.59944 -> 0.6; via_drill 0.39878 -> 0.4
- rule trace_min: 0.254 -> 0.19
- rule via_min_drill: 0.35052 -> 0.25
- rule via_min_size: 0.398 -> 0.58
- board text added: "20mm X 20mm Heatsink"
- board text added: "Board design improved by Bob808 oct.2018"
- board text added: "CERN OSH License 1.2"
- board text added: "E0"
- board text added: "E1"
- board text added: "Sweet Silence!"
- board text added: "V1.0"
- board text added: "X-AXIS"
- board text added: "Y-AXIS"
- board text added: "Z-AXIS"
- board text removed: "DUET 2"
- board text removed: "Designed and assembled in the UK"
- board text removed: "Duet2 V1.04 Design: David Crocker: www.escher3d.com Tony Lock: www.think3dprint3d.com CERN OSH License 1.2"
- board text removed: "E0 MOTOR"
- board text removed: "E0_STEP E0_DIR E0_EN/CS"
- board text removed: "E1 MOTOR"
- board text removed: "E1_STEP E1_DIR E1_EN/CS"
- board text removed: "X-AXIS MOTOR"
- board text removed: "X_STEP X_DIR X_EN/CS"
- board text removed: "Y-AXIS MOTOR"
- board text removed: "Y_STEP Y_DIR Y_EN/CS"
- board text removed: "Z-AXIS MOTOR"
- board text removed: "Z_STEP Z_DIR Z_EN/CS"
- board text removed: "www.duet3d.com"

Commit message: Add files via upload
Other:
- board text added: "10mm X 10mm Heatsink"
- board text removed: "20mm X 20mm Heatsink"
Changed lines of the file:
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@@
   )
   (layers
-    (0 Front mixed hide)
-    (1 Inner3 signal hide)
+    (0 Front mixed)
+    (1 Inner3 signal)
     (2 Inner2 power hide)
-    (31 Back power hide)
+    (31 Back power)
     (35 F.Paste user hide)
     (36 B.SilkS user)
-    (37 F.SilkS user hide)
+    (37 F.SilkS user)
     (38 B.Mask user hide)
     (39 F.Mask user hide)
@@
     (effects (font (size 1.524 1.524) (thickness 0.2) italic))
   )
-  (gr_text "20mm X 20mm Heatsink" (at 102.936 44.96198) (layer F.SilkS)
+  (gr_text "10mm X 10mm Heatsink" (at 102.936 44.96198) (layer F.SilkS)
     (effects (font (size 0.5 0.5) (thickness 0.1)))
   )
-  (gr_text "20mm X 20mm Heatsink" (at 100.015 63.50398) (layer F.SilkS)
+  (gr_text "10mm X 10mm Heatsink" (at 100.015 63.50398) (layer F.SilkS)
     (effects (font (size 0.5 0.5) (thickness 0.1)))
   )
-  (gr_text "20mm X 20mm Heatsink" (at 100.2055 78.74398) (layer F.SilkS)
+  (gr_text "10mm X 10mm Heatsink" (at 100.2055 78.74398) (layer F.SilkS)
     (effects (font (size 0.5 0.5) (thickness 0.1)))
   )
-  (gr_text "20mm X 20mm Heatsink" (at 100.269 95.19048) (layer F.SilkS)
+  (gr_text "10mm X 10mm Heatsink" (at 100.269 95.19048) (layer F.SilkS)
     (effects (font (size 0.5 0.5) (thickness 0.1)))
   )
-  (gr_text "20mm X 20mm Heatsink" (at 100.2055 112.39898) (layer F.SilkS)
+  (gr_text "10mm X 10mm Heatsink" (at 100.2055 112.39898) (layer F.SilkS)
     (effects (font (size 0.5 0.5) (thickness 0.1)))
   )

Commit message: fixed DRC
FIxed DRC errors.
Parts:
- moved Ju1 0.19 mm to (94.2, 127.6)
- moved C105 0.19 mm to (94.2, 130.6)
Routing:
- net Net-(L25-Pad2): track 46.2 -> 49.4 mm
Changed lines of the file:
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@@
     (thickness 1.6002)
     (drawings 374)
-    (tracks 10011)
+    (tracks 10021)
     (zones 0)
     (modules 430)
@@
   (layers
     (0 Front mixed)
-    (1 Inner3 signal)
+    (1 Inner3 signal hide)
     (2 Inner2 power hide)
-    (31 Back power)
+    (31 Back power hide)
     (35 F.Paste user hide)
-    (36 B.SilkS user)
+    (36 B.SilkS user hide)
     (37 F.SilkS user)
     (38 B.Mask user hide)
@@
   )
   (module complib:C_0603 (layer Front)
-    (at 94.427 130.55998 270)
+    (at 94.234 130.556 270)
     (descr "SMT capacitor, 0603")
     (fp_text reference C105 (at 0.127 -1.2065 270) (layer F.SilkS)
@@
   )
   (module complib:R_0603 (layer Front)
-    (at 94.427 127.57548 90)
+    (at 94.234 127.5588 90)
     (attr smd)
     (fp_text reference Ju1 (at 0.0508 1.0922 90) (layer F.SilkS) hide
@@
   (segment (start 98.7725 130.90748) (end 96.7765 130.87748) (width 0.381) (layer Back) (net 67))
   (segment (start 103.317 124.08298) (end 103.317 124.46398) (width 0.4455) (layer Front) (net 67))
-  (via (at 95.443 128.34747) (size 0.6) (drill 0.4) (layers Front Back) (net 67))
-  (via (at 95.443 129.54398) (size 0.6) (drill 0.4) (layers Front Back) (net 67))
+  (via (at 95.3008 129.4892) (size 0.6) (drill 0.4) (layers Front Back) (net 67))
   (segment (start 101.122 130.90748) (end 102.596952 130.90748) (width 0.4455) (layer Front) (net 67))
   (segment (start 101.122 130.90748) (end 100.172 130.90748) (width 0.381) (layer Front) (net 67))
@@
   (segment (start 97.572 130.90748) (end 98.872 129.60748) (width 0.381) (layer Front) (net 67))
   (segment (start 96.622 130.90748) (end 97.572 130.90748) (width 0.381) (layer Front) (net 67))
+  (via (at 95.4532 128.14587) (size 0.6) (drill 0.4) (layers Front Back) (net 67))
   (segment (start 144.566639 117.078761) (end 144.26692 117.37848) (width 0.254) (layer Front) (net 68))
   (segment (start 145.553855 117.078761) (end 144.566639 117.078761) (width 0.254) (layer Front) (net 68))
@@
   (segment (start 89.474001 128.210481) (end 90.236 128.97248) (width 0.254) (layer Front) (net 284))
   (segment (start 95.8494 125.86098) (end 95.12042 125.86098) (width 0.254) (layer Front) (net 284))
-  (segment (start 94.81308 129.23156) (end 94.554 128.97248) (width 0.381) (layer Front) (net 284))
-  (segment (start 94.554 128.97248) (end 94.808 128.97248) (width 0.381) (layer Front) (net 284))
+  (segment (start 94.6404 128.6256) (end 94.38132 128.36652) (width 0.381) (layer Front) (net 284))
+  (segment (start 94.3356 128.6764) (end 94.5896 128.6764) (width 0.381) (layer Front) (net 284))
   (segment (start 94.554 128.50258) (end 94.427 128.37558) (width 0.381) (layer Front) (net 284))
   (segment (start 94.554 128.97248) (end 94.554 128.50258) (width 0.381) (layer Front) (net 284))
@@
   (segment (start 88.966 127.70248) (end 90.236 128.97248) (width 0.381) (layer Front) (net 284))
   (segment (start 88.966 125.996778) (end 88.966 127.70248) (width 0.381) (layer Front) (net 284))
-  (segment (start 96.082 128.97248) (end 94.554 128.97248) (width 0.25) (layer Front) (net 284))
-  (segment (start 96.097 128.95748) (end 96.082 128.97248) (width 0.25) (layer Front) (net 284))
   (segment (start 96.622 128.95748) (end 96.097 128.95748) (width 0.25) (layer Front) (net 284))
+  (segment (start 96.097 128.95748) (end 95.9104 128.77088) (width 0.25) (layer Front) (net 284))
+  (segment (start 95.9104 128.77088) (end 94.7556 128.77088) (width 0.25) (layer Front) (net 284))
+  (segment (start 94.7556 128.77088) (end 94.554 128.97248) (width 0.25) (layer Front) (net 284))
   (segment (start 94.1095 134.05248) (end 94.4016 134.34458) (width 0.381) (layer Front) (net 285))
   (segment (start 90.236 134.05248) (end 94.1095 134.05248) (width 0.381) (layer Front) (net 285))
@@
   (segment (start 93.792 120.46348) (end 93.792 120.20948) (width 0.254) (layer Back) (net 287))
   (segment (start 93.991 120.65818) (end 93.991 120.64548) (width 0.254) (layer Back) (net 287))
-  (segment (start 92.7506 121.89858) (end 93.991 120.65818) (width 0.254) (layer Back) (net 287))
+  (segment (start 92.7506 121.8396) (end 93.991 120.5992) (width 0.254) (layer Back) (net 287))
   (segment (start 92.7506 121.92398) (end 92.7506 121.89858) (width 0.254) (layer Back) (net 287))
   (segment (start 92.7506 121.92398) (end 92.7506 121.63188) (width 0.254) (layer Back) (net 287))
@@
   (segment (start 93.2475 123.76548) (end 93.2475 122.91298) (width 0.254) (layer Back) (net 321))
   (segment (start 93.552581 122.607899) (end 93.552581 122.49548) (width 0.254) (layer Back) (net 321))
-  (segment (start 93.2475 122.91298) (end 93.552581 122.607899) (width 0.254) (layer Back) (net 321))
+  (segment (start 93.319319 122.936281) (end 93.6244 122.6312) (width 0.254) (layer Back) (net 321))
   (segment (start 93.552581 122.49548) (end 93.552581 122.861899) (width 0.254) (layer Back) (net 321))
   (segment (start 93.552581 121.738665) (end 93.552581 122.49548) (width 0.254) (layer Back) (net 321))
@@
   (segment (start 93.665 121.86048) (end 93.665 122.36848) (width 0.254) (layer Back) (net 321))
   (segment (start 93.665 122.36848) (end 93.665 122.58598) (width 0.254) (layer Back) (net 321))
-  (segment (start 93.2475 123.76548) (end 94.046 122.96698) (width 0.254) (layer Back) (net 321))
   (segment (start 93.9825 121.66998) (end 93.919 121.60648) (width 0.254) (layer Back) (net 321))
   (segment (start 93.9825 123.06698) (end 93.9825 121.66998) (width 0.254) (layer Back) (net 321))
@@
   (segment (start 96.9035 118.67268) (end 96.9035 118.62198) (width 0.254) (layer Back) (net 321))
   (segment (start 96.9035 118.62198) (end 97.1575 118.36798) (width 0.254) (layer Back) (net 321))
+  (segment (start 93.2475 123.10798) (end 93.36868 122.9868) (width 0.25) (layer Back) (net 321))
+  (segment (start 93.2475 124.08298) (end 93.2475 123.10798) (width 0.25) (layer Back) (net 321))
+  (segment (start 93.82298 122.9868) (end 93.92458 123.0884) (width 0.25) (layer Back) (net 321))
+  (segment (start 93.36868 122.9868) (end 93.82298 122.9868) (width 0.25) (layer Back) (net 321))
+  (segment (start 93.92458 123.0884) (end 94.046 122.96698) (width 0.254) (layer Back) (net 321))
+  (segment (start 93.2475 124.08298) (end 93.2475 123.3129) (width 0.25) (layer Back) (net 321))
+  (segment (start 93.4212 123.1392) (end 93.87378 123.1392) (width 0.25) (layer Back) (net 321))
+  (segment (start 93.2475 123.3129) (end 93.4212 123.1392) (width 0.25) (layer Back) (net 321))
+  (segment (start 93.87378 123.1392) (end 93.92458 123.0884) (width 0.254) (layer Back) (net 321))
+  (segment (start 93.2475 123.76548) (end 93.87378 123.1392) (width 0.254) (layer Back) (net 321))
   (segment (start 94.1815 117.24348) (end 93.184 118.24098) (width 0.25) (layer Back) (net 322))
   (segment (start 93.184 118.24098) (end 93.2205 118.24098) (width 0.254) (layer Back) (net 322))

Commit message: Update Duet2/Duet2v1.04/DuetWifi.kicad_pcb
Other:
- board text added: "“Based on the DuetWifi by Think3dPrint3d and Esher3d, see www.duet3d.com for the original DuetWifi information. This reproduction/ modification is not endorsed or supported in any way by Think3dPrint3d or Escher3d”"
Changed lines of the file:
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@@
   (general
     (thickness 1.6002)
-    (drawings 374)
+    (drawings 375)
     (tracks 10021)
     (zones 0)
@@
   )
   (layers
-    (0 Front mixed)
+    (0 Front mixed hide)
     (1 Inner3 signal hide)
     (2 Inner2 power hide)
     (31 Back power hide)
     (35 F.Paste user hide)
-    (36 B.SilkS user hide)
-    (37 F.SilkS user)
+    (36 B.SilkS user)
+    (37 F.SilkS user hide)
     (38 B.Mask user hide)
     (39 F.Mask user hide)
@@
     )
   )
+  (gr_text "“Based on the DuetWifi by Think3dPrint3d and Esher3d, see \nwww.duet3d.com for the original DuetWifi information. This reproduction/\nmodification is not endorsed or supported in any way by Think3dPrint3d \nor Escher3d”" (at 113.2332 96.6724 270) (layer B.SilkS)
+    (effects (font (size 1 1) (thickness 0.1)) (justify mirror))
+  )
   (gr_text "CERN OSH License 1.2 " (at 131.2672 103.0732 90) (layer F.SilkS)
